File: chute_release.kicad_pcb (KiCad board)
At the start: 4 copper layers, 22.3 x 37.7 mm, 37 parts, among them J1 Conn_01x02, J2 Conn_01x03, J3 USB4105-GF-A, U1 NCP1117-3.3_SOT223, U2 W25Q128JVS, U3 RP2040, U4 DPS310XTSA1, Y1 ABM8-272-T3

Commit message: WIP - Started implementation of selector switch
Parts:
- removed J1: Conn_01x02, Connector_PinHeader_2.54mm:PinHeader_1x02_P2.54mm_Vertical
- added C20: 100n, Capacitor_SMD:C_0402_1005Metric, B.Cu at (117.2, 102.4)
- added C21: 100n, Capacitor_SMD:C_0402_1005Metric, B.Cu at (128.6, 105.2)
- added CR1: TLMS1100-GS08, duso:LED_VISHAY_TLMX1100_VIS, B.Cu at (124.7, 87.4)
- added D1: MBR0540, Diode_SMD:D_SOD-123, B.Cu at (117.9, 91.7)
- added D2: 1N4148WS, Diode_SMD:D_SOD-323, F.Cu at (107.5, 103.9)
- added J4: USB4105-GF-A, duso:GCT_USB4105-GF-A, F.Cu at (124.8, 83.7)
- added Q1: DMG3415UFY4Q-7, duso:TRANS_DMG3415UFY4Q-7, B.Cu at (120.1, 92.7)
- added R11: 5k, Resistor_SMD:R_0603_1608Metric, B.Cu at (121.1, 86.1)
- added R12: 10k, Resistor_SMD:R_0603_1608Metric, B.Cu at (121.8, 83.4)
- added R13: 10k, Resistor_SMD:R_0603_1608Metric, B.Cu at (127.0, 83.5)
- added R14: 10k, Resistor_SMD:R_0402_1005Metric, F.Cu at (113.6, 105.9)
- added SW1: SH-7050TB, duso:SH-7050B_NDC, F.Cu at (124.8, 93.4)
- added SW2: SW_Push, duso:NanoT-AS, F.Cu at (126.0, 100.3)
- added SW3: SW_Push, duso:NanoT-AS, F.Cu at (123.5, 100.3)
- added U5: MCP73831-2-OT, Package_TO_SOT_SMD:SOT-23-5, B.Cu at (124.4, 83.9)
- C1, C10, C11, C12, C14, C15, C16, C18, C19, C2, C6, C7, C8, C9, R3, R4, R5, R6, R7, R8, R9, U2, U3, U4, Y1: moved to B.Cu
- C13: value 100n -> 4.7u; moved to B.Cu
- C17: value 100n -> 10u; moved to B.Cu
- C3, C4: value 10u -> 4.7u; footprint Capacitor_SMD:C_0805_2012Metric -> Capacitor_SMD:C_0402_1005Metric
- J3: value USB4105-GF-A -> Conn_01x02_Pin; footprint duso:GCT_USB4105-GF-A -> Connector_JST:JST_PH_B2B-PH-K_1x02_P2.00mm_Vertical
- R10: value 5k -> 10k; moved to B.Cu
- R2: value DNF -> 10k; moved to B.Cu
- U1: value NCP1117-3.3_SOT223 -> AP7361C-33E
- moved R1 35.7 mm to (107.4, 102.3), turned to 180 degrees
- moved C12 34.9 mm to (118.3, 105.5), turned to 90 degrees
- moved C15 34.2 mm to (118.3, 110.3), turned to -90 degrees
- moved C11 32.5 mm to (118.2, 102.4)
- moved C9 30.7 mm to (119.2, 102.4)
- moved R5 29.0 mm to (120.2, 102.4)
- moved R10 27.9 mm to (118.4, 94.6), turned to 0 degrees
- moved R4 27.3 mm to (121.2, 102.4)
- moved R2 27.0 mm to (132.9, 105.1), turned to 90 degrees
- moved C10 26.3 mm to (122.3, 102.4)
- moved C3 25.9 mm to (120.7, 90.3), turned to -90 degrees
- moved C8 25.7 mm to (122.4, 114.6)
- moved C13 25.6 mm to (123.3, 86.1), turned to 180 degrees
- moved C2 25.2 mm to (128.2, 115.3), turned to -90 degrees
- moved C7 24.8 mm to (123.3, 102.4)
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Connections:
- C17 pad 1: +3V3 -> +BATT
- C3 pad 1: VBUS -> Net-(D1-K)
- R1 pad 2: /MCU/~{USB_BOOT} -> Net-(D2-A)
- R10 pad 1: Net-(J3-CC2) -> VBUS
- R9 pad 1: Net-(J3-CC1) -> Net-(J4-CC1)
- U1 pad 1: GND -> Net-(D1-K)
- U1 pad 2: +3V3 -> GND
- U1 pad 3: VBUS -> +3V3
- U3 pad 34: /MCU/GPIO22 -> HEX_SW_1
- U3 pad 35: /MCU/GPIO23 -> HEX_SW_2
- U3 pad 36: /MCU/GPIO24 -> HEX_SW_4
- U3 pad 37: /MCU/GPIO25 -> HEX_SW_8
Routing:
- net GND: track 48.1 -> 0.00 mm, vias 35 -> 0
- net /MCU/GPIO0: track 27.8 -> 0.00 mm
- net +1V1: track 27.8 -> 8.82 mm, vias 2 -> 0
- net +3V3: track 48.7 -> 33.8 mm, vias 9 -> 0
- net USB_D+: track 12.1 -> 0.00 mm
- net USB_D-: track 11.3 -> 0.00 mm
- net SDI: track 12.9 -> 3.39 mm
- net /MCU/QSPI_SS: track 23.8 -> 15.2 mm
- net Net-(D1-K): track 0.00 -> 8.25 mm
- net /MCU/XIN: track 17.6 -> 9.37 mm
- net SDK: track 12.8 -> 5.35 mm
- net Net-(J3-CC1): track 6.12 -> 0.00 mm
- net Net-(J3-CC2): track 5.71 -> 0.00 mm
- net Net-(C2-Pad1): track 10.9 -> 5.41 mm
- net Net-(J4-CC1): track 0.00 -> 5.32 mm, vias 0 -> 1
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Other:
- board size 22.3 x 37.7 mm -> 19.3 x 28.2 mm
