File: chute_release.kicad_sch (KiCad schematic)
At the start: 0 parts

Commit message: WIP - Started implementation of selector switch
Other:
- added sheet INTERFACE (interface.kicad_sch)
Changed lines of the file:
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@@
+	)
+	(sheet
+		(at 165.1 87.63)
+		(size 106.68 44.45)
+		(fields_autoplaced yes)
+		(stroke
+			(width 0.1524)
+			(type solid)
+		)
+		(fill
+			(color 0 0 0 0.0000)
+		)
+		(property "Sheetname" "INTERFACE"
+			(at 165.1 86.9184 0)
+			(effects
+				(font
+					(size 1.27 1.27)
+				)
+				(justify left bottom)
+			)
+		)
+		(property "Sheetfile" "interface.kicad_sch"
+			(at 165.1 132.6646 0)
+			(effects
+				(font
+					(size 1.27 1.27)
+				)
+				(justify left top)
+			)
+		)
+		(instances
+			(project "chute_release"
+				(path "/9d05c756-443f-4d4d-9854-905483bdebb5"
+					(page "5")
+				)
+			)
+		)
 	)
 	(sheet
