File: mcu.kicad_sch (KiCad schematic)
At the start: 17 parts, among them J1 Conn_01x02, J2 Conn_01x03, U2 W25Q128JVS, U3 RP2040, Y1 ABM8-272-T3

Commit message: WIP - Started implementation of selector switch
Parts:
- removed J1: Conn_01x02, Connector_PinHeader_2.54mm:PinHeader_1x02_P2.54mm_Vertical, symbol Connector_Generic:Conn_01x02
- added D2: 1N4148WS, Diode_SMD:D_SOD-323, symbol Diode:1N4148WS
- added R14: 10k, Resistor_SMD:R_0402_1005Metric, symbol Device:R
- added SW2, SW3: SW_Push, duso:NanoT-AS, symbol Switch:SW_Push
- R2: value DNF -> 10k; now fitted
Connections:
- net +3V3: now also R14.1
- net GND: now also SW2.2, SW3.2
- net RUN: now also R14.2, SW3.1
- net GPIO22 renamed HEX_SW_1
- net GPIO23 renamed HEX_SW_2
- net GPIO24 renamed HEX_SW_4
- net GPIO25 renamed HEX_SW_8
- net ~{USB_BOOT}: no longer names the net of R1.2
- net ~{USB_BOOT}: now also D2.2 (A)
- new net: D2.1 (K), SW2.1
Other:
- moved on the sheet: C1, C2, C6, R3, U2, Y1
